File: pcb/v1/sfp_moduloIC.kicad_sch (KiCad schematic)
At the start: 157 parts, among them J1 SPI, J2 FTDI, J3 SWD, J4 RATE, J5 DIS, J6 SFP, J7 POWER, J8 IN, Q1 AO3401A, Q2 BC848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

Commit message: v4.1
Parts:
- L2, L3: JLCPCB Part # C18734508 -> C41902
Changed lines of the file:
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@@
 			)
 		)
-		(property "JLCPCB Part #" "C18734508"
+		(property "JLCPCB Part #" "C41902"
 			(at 377.19 218.44 90)
 			(effects
@@
 			)
 		)
-		(property "JLCPCB Part #" "C18734508"
+		(property "JLCPCB Part #" "C41902"
 			(at 347.98 218.44 90)
 			(effects
