File: pcb/v2/sfp_moduloIC.kicad_sch (KiCad schematic)
At the start: 154 parts, among them J1 SPI, J2 FTDI, J3 SWD, J4 RATE, J5 DIS, J6 SFP, J7 POWER, J8 IN, Q1 BC848, Q2 BC848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

Commit message: v4.1
Parts:
- removed H2: FIX, MountingHole:MountingHole_3.2mm_M3_Pad, symbol Mechanical:MountingHole_Pad
- added J11: ANT, KiCad3:CONUFL001SMDT, symbol Connector:Conn_Coaxial_Small
- added JP1, JP2: SEL, Jumper:SolderJumper-3_P1.3mm_Open_RoundedPad1.0x1.5mm, symbol Jumper:SolderJumper_3_Open
- L2, L3: JLCPCB Part # C18734508 -> C41902
- renumbered H3 to H2
Connections:
- net +3V3: now also JP1.3 (B), JP2.3 (B); no longer R34.1, R35.1, R36.1, R37.1, R38.1, R39.1, R40.1, R41.1, R42.1, R43.1
- net ANT: now also J11.1 (In)
- net GND: now also J11.2 (Ext), J11.3 (arm), JP1.1 (A), JP2.1 (A)
- new net CONFIG: JP2.2 (C), R35.1, R36.1, R37.1, R38.1, R40.1, R41.1, R42.1, R43.1
- new net DISAUTO: JP1.2 (C), R34.1, R39.1
Other:
- moved on the sheet: H1, H2
